File: kicad/alu/alu4.sch (KiCad schematic (older format))
At the start: 15 parts, among them U11 74LS283, U12 74LS157, U13 74LS86, U14 74LS86, U15 74LS86, U7 74LS08, U8 74LS08, U9 74LS08

Commit message: update
Parts:
- added C22: C, Capacitor_THT:C_Disc_D5.0mm_W2.5mm_P2.50mm, symbol Device:C
Connections:
- net GND: now also C22.1
- net VCC: now also C22.2
