File: kicad/alu/alu.kicad_pcb (KiCad board)
At the start: 2 copper layers, 237.5 x 102.9 mm, 89 parts, among them J1 Conn_02x30_Counter_Clockwise, J2 Conn_01x09_Male, J3 Conn_01x09_Male, J4 Conn_01x09_Male, J5 Conn_01x03_Male, J6 Conn_01x03_Male, J7 Conn_01x02_Male, U1 74LS377, U10 74LS32, U11 74LS283, U12 74LS157, U13 74LS86, U14 74LS86, U15 74LS86, U16 74LS08, U17 74LS08, U18 74LS86, U19 74LS86, U2 74LS377, U20 74LS08, U21 74LS283, U22 74LS157, U23 74LS86, U3 74LS244, U4 74LS377, U5 74LS32, U6 74LS02, U7 74LS08, U8 74LS08, U9 74LS08

Commit message: update
Parts:
- removed the REF** at (261.6, 139.7)
- removed the REF** at (261.6, 47.0)
- added C22: C, Capacitor_THT:C_Disc_D5.0mm_W2.5mm_P2.50mm, F.Cu at (67.3, 113.0)
- added C23: C, Capacitor_THT:C_Disc_D5.0mm_W2.5mm_P2.50mm, F.Cu at (67.3, 132.1)
- added REF**: MountingHole_3.2mm_M3, MountingHole:MountingHole_3.2mm_M3, F.Cu at (261.6, 137.2)
- added REF**: MountingHole_3.2mm_M3, MountingHole:MountingHole_3.2mm_M3, F.Cu at (261.6, 49.5)
- moved J7 254.4 mm to (55.9, 64.8)
- moved J6 246.5 mm to (71.6, 64.0), turned to 180 degrees
- moved C3 233.4 mm to (115.6, 100.4), turned to 270 degrees
- moved C1 232.0 mm to (67.3, 94.0), turned to 270 degrees
- moved U23 219.0 mm to (111.8, 97.8)
- moved U22 213.5 mm to (111.8, 114.3)
- moved C7 212.7 mm to (114.3, 50.8), turned to 270 degrees
- moved U21 210.6 mm to (111.8, 130.8)
- moved C4 199.6 mm to (114.3, 67.3), turned to 270 degrees
- moved U19 192.9 mm to (188.0, 130.8)
- moved C2 191.8 mm to (114.3, 83.8), turned to 270 degrees
- moved C6 190.8 mm to (115.6, 116.8), turned to 270 degrees
- moved C5 173.7 mm to (115.6, 133.4), turned to 270 degrees
- moved U18 162.5 mm to (151.1, 104.1)
- moved C20 158.1 mm to (154.9, 57.2), turned to 270 degrees
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Routing:
- net D7h: track 0.00 -> 336.1 mm, vias 0 -> 4
- net D6h: track 0.00 -> 334.5 mm, vias 0 -> 5
- net E1: track 0.00 -> 303.4 mm, vias 0 -> 6
- net LT: track 0.00 -> 302.7 mm, vias 0 -> 6
- net E0: track 0.00 -> 292.7 mm, vias 0 -> 8
- net Z: track 0.00 -> 287.9 mm, vias 0 -> 5
- net E2: track 0.00 -> 278.9 mm, vias 0 -> 6
- net E3: track 0.00 -> 277.3 mm, vias 0 -> 8
- net D0h: track 0.00 -> 266.2 mm, vias 0 -> 3
- net D1h: track 0.00 -> 263.8 mm, vias 0 -> 2
- net D2h: track 0.00 -> 259.0 mm, vias 0 -> 3
- net CLK: track 0.00 -> 258.6 mm, vias 0 -> 1
- net D3h: track 0.00 -> 258.2 mm, vias 0 -> 4
- net GND: track 0.00 -> 255.9 mm, vias 0 -> 17
- net NY: track 0.00 -> 253.7 mm, vias 0 -> 7
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- added copper zone on F.Cu, net GND
- added copper zone on B.Cu, net VCC
Other:
- board text added: "SCAMP ALU Card by jes"
- board text removed: "SCAMP ALU Card"

Commit message: Update PCB
Parts:
- moved J1 0.40 mm to (34.3, 56.5)
Routing:
- net GND: track 255.9 -> 298.6 mm, vias 17 -> 18
- net VCC: track 71.8 -> 85.4 mm, vias 5 -> 7
- net CLK: track 258.6 -> 252.4 mm
- net Net-(U21-Pad13): track 26.3 -> 21.6 mm, vias 2 -> 0
- net ~YI~: track 223.6 -> 219.1 mm, vias 7 -> 5
- net Net-(U20-Pad11): track 49.1 -> 45.5 mm
- net Z: track 287.9 -> 284.7 mm, vias 5 -> 3
- net LT: track 302.7 -> 300.4 mm, vias 6 -> 4
- net D3h: track 258.2 -> 255.9 mm, vias 4 -> 0
- net nz2: track 71.3 -> 73.0 mm, vias 2 -> 1
- net Net-(U18-Pad11): track 74.2 -> 72.6 mm, vias 2 -> 1
- net Net-(U12-Pad9): track 20.1 -> 18.6 mm, vias 2 -> 0
- net Net-(U14-Pad1): track 20.1 -> 18.6 mm, vias 2 -> 0
- net Net-(U19-Pad3): track 94.3 -> 92.9 mm, vias 3 -> 1
- net D13: track 16.5 -> 15.1 mm, vias 2 -> 1
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Other:
- board text added: "D0"
- board text added: "D1"
- board text added: "D10"
- board text added: "D11"
- board text added: "D12"
- board text added: "D13"
- board text added: "D14"
- board text added: "D15"
- board text added: "D2"
- board text added: "D3"
- board text added: "D4"
- board text added: "D5"
- board text added: "D6"
- board text added: "D7"
- board text added: "D8"
- board text added: "D9"
- board text added: "GND"
- board text added: "In"
- board text added: "LT"
- board text added: "Out"
- board text added: "Result"
- board text added: "X Register"
- board text added: "Y Register"
- board text added: "Z"
- board text added: "carry"
- board text added: "nz"

Commit message: Fix unconnected nets
Routing:
- net GND: track 298.6 -> 331.3 mm, vias 18 -> 23
Changed lines of the file:
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@@
     (thickness 1.6)
     (drawings 33)
-    (tracks 1941)
+    (tracks 1956)
     (zones 0)
     (modules 91)
@@
   (segment (start 170.18 104.14) (end 168.91 104.14) (width 0.25) (layer F.Cu) (net 2))
   (segment (start 167.64 102.87) (end 167.64 100.33) (width 0.25) (layer B.Cu) (net 2))
-  (segment (start 37.594999 94.485001) (end 47.514999 94.485001) (width 0.25) (layer F.Cu) (net 2))
   (segment (start 47.514999 94.485001) (end 48.5 93.5) (width 0.25) (layer F.Cu) (net 2))
   (via (at 48.5 93.5) (size 0.8) (drill 0.4) (layers F.Cu B.Cu) (net 2))
@@
   (segment (start 173.99 49.53) (end 173.99 53.34) (width 0.25) (layer B.Cu) (net 2))
   (segment (start 172.72 48.26) (end 173.99 49.53) (width 0.25) (layer B.Cu) (net 2))
+  (via (at 45.72 95.25) (size 0.8) (drill 0.4) (layers F.Cu B.Cu) (net 2))
+  (segment (start 45.214999 94.744999) (end 45.72 95.25) (width 0.25) (layer F.Cu) (net 2))
+  (segment (start 45.214999 94.485001) (end 45.214999 94.744999) (width 0.25) (layer F.Cu) (net 2))
+  (segment (start 37.594999 94.485001) (end 45.214999 94.485001) (width 0.25) (layer F.Cu) (net 2))
+  (segment (start 45.214999 94.485001) (end 47.514999 94.485001) (width 0.25) (layer F.Cu) (net 2))
+  (segment (start 45.72 95.25) (end 45.72 102.87) (width 0.25) (layer B.Cu) (net 2))
+  (segment (start 45.72 102.87) (end 48.26 102.87) (width 0.25) (layer B.Cu) (net 2))
+  (via (at 107.95 77.47) (size 0.8) (drill 0.4) (layers F.Cu B.Cu) (net 2))
+  (segment (start 107.95 72.39) (end 107.95 77.47) (width 0.25) (layer B.Cu) (net 2))
+  (via (at 100.33 77.47) (size 0.8) (drill 0.4) (layers F.Cu B.Cu) (net 2))
+  (segment (start 107.95 77.47) (end 100.33 77.47) (width 0.25) (layer F.Cu) (net 2))
+  (segment (start 100.33 77.47) (end 97.79 77.47) (width 0.25) (layer B.Cu) (net 2))
+  (via (at 97.79 77.47) (size 0.8) (drill 0.4) (layers F.Cu B.Cu) (net 2))
+  (via (at 91.44 77.47) (size 0.8) (drill 0.4) (layers F.Cu B.Cu) (net 2))
+  (segment (start 97.79 77.47) (end 91.44 77.47) (width 0.25) (layer F.Cu) (net 2))
   (segment (start 43.7 53.95) (end 44.45 53.95) (width 0.25) (layer F.Cu) (net 3))
   (segment (start 38.200002 53.95) (end 43.7 53.95) (width 0.25) (layer F.Cu) (net 3))
@@
   (segment (start 182.222999 77.365001) (end 182.88 78.022002) (width 0.25) (layer F.Cu) (net 159))
   (segment (start 182.88 78.232) (end 182.88 81.28) (width 0.25) (layer F.Cu) (net 159))
-  (segment (start 97.79 78.486) (end 97.79 81.28) (width 0.25) (layer F.Cu) (net 159))
-  (segment (start 99.568 76.708) (end 97.79 78.486) (width 0.25) (layer F.Cu) (net 159))
-  (segment (start 148.844 76.708) (end 99.568 76.708) (width 0.25) (layer F.Cu) (net 159))
+  (segment (start 97.79 80.14863) (end 97.79 81.28) (width 0.25) (layer F.Cu) (net 159))
+  (segment (start 148.844 76.708) (end 99.625002 76.708) (width 0.25) (layer F.Cu) (net 159))
+  (segment (start 99.625002 76.708) (end 97.79 78.543002) (width 0.25) (layer F.Cu) (net 159))
+  (segment (start 97.79 78.543002) (end 97.79 80.14863) (width 0.25) (layer F.Cu) (net 159))
   (via (at 133.096 74.676) (size 0.8) (drill 0.4) (layers F.Cu B.Cu) (net 160))
   (segment (start 99.06 74.676) (end 133.096 74.676) (width 0.25) (layer F.Cu) (net 160))

Commit message: Tidy up ALU card
Parts:
- moved C1 175.4 mm to (238.8, 57.2)
- moved C10 175.1 mm to (67.3, 96.5)
- moved C21 146.0 mm to (115.6, 135.5), turned to 90 degrees
- moved C4 139.1 mm to (238.8, 129.5)
- moved C11 125.1 mm to (115.6, 86.4)
- moved C2 124.5 mm to (238.8, 83.8), turned to 90 degrees
- moved C3 123.3 mm to (238.8, 105.5)
- moved C12 90.9 mm to (115.6, 67.3)
- moved C18 86.9 mm to (154.9, 106.7), turned to 270 degrees
- moved C7 77.5 mm to (191.8, 50.8)
- moved C20 72.3 mm to (154.9, 129.5), turned to 90 degrees
- moved C15 68.4 mm to (115.6, 50.8)
- moved C23 56.3 mm to (115.5, 103.0), turned to 90 degrees
- moved C17 54.8 mm to (191.8, 116.8)
- moved C5 52.4 mm to (67.3, 113.1)
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Routing:
- net GND: track 331.3 -> 391.9 mm, vias 23 -> 30
- net VCC: track 85.4 -> 104.2 mm, vias 7 -> 5
- net Net-(U11-Pad12): track 71.4 -> 67.7 mm, vias 1 -> 0
- net Net-(U12-Pad5): track 46.9 -> 44.2 mm, vias 2 -> 1
- net Net-(U12-Pad14): track 47.7 -> 45.1 mm
- net Net-(U11-Pad10): track 25.2 -> 22.7 mm, vias 2 -> 1
- net E0: track 292.4 -> 294.5 mm, vias 7 -> 8
- net Net-(U12-Pad11): track 44.6 -> 42.7 mm
- net NO: track 158.0 -> 159.7 mm
- net Net-(U11-Pad13): track 23.2 -> 21.6 mm
- net carry_in: track 36.6 -> 37.8 mm
- net Net-(U12-Pad7): track 22.4 -> 21.2 mm, vias 2 -> 1
- net Net-(U12-Pad12): track 19.8 -> 18.6 mm, vias 2 -> 0
- net Net-(U11-Pad1): track 29.8 -> 30.9 mm
- net /aluhigh/C_in: track 45.0 -> 46.0 mm
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Other:
- board text added: "Adder"
- board text added: "And"
- board text added: "EX"
- board text added: "EY"
- board text added: "Flags register"
- board text added: "High nybble ALU"
- board text added: "Low nybble ALU"
- board text added: "Mux"
- board text added: "NO"
- board text added: "NX"
- board text added: "NY"
- board text added: "Result buffer"
- board text added: "X register"
- board text added: "Y register"
- board text added: "Zero detection"
- board text removed: "X Register"
- board text removed: "Y Register"
