File: kicad/alu/alu.kicad_pcb (KiCad board)
At the start: 2 copper layers, 237.5 x 102.9 mm, 91 parts, among them J1 Conn_02x30_Counter_Clockwise, J2 Conn_01x09_Male, J3 Conn_01x09_Male, J4 Conn_01x09_Male, J5 Conn_01x03_Male, J6 Conn_01x03_Male, J7 Conn_01x02_Male, U1 74LS377, U10 74LS32, U11 74LS283, U12 74LS157, U13 74LS86, U14 74LS86, U15 74LS86, U16 74LS08, U17 74LS08, U18 74LS86, U19 74LS86, U2 74LS377, U20 74LS08, U21 74LS283, U22 74LS157, U23 74LS86, U3 74LS244, U4 74LS377, U5 74LS32, U6 74LS02, U7 74LS08, U8 74LS08, U9 74LS08

Commit message: Tidy up ALU card slightly
Routing:
- net carry_in: track 37.8 -> 33.8 mm, vias 2 -> 1
- net D5h: track 228.6 -> 224.8 mm, vias 3 -> 1
- net ~YI~: track 219.1 -> 216.4 mm, vias 5 -> 2
- net Y1: track 81.4 -> 79.1 mm, vias 2 -> 1
- net Net-(U11-Pad11): track 93.9 -> 91.9 mm
- net Net-(U12-Pad7): track 21.2 -> 23.1 mm, vias 1 -> 0
- net Net-(U11-Pad2): track 77.6 -> 75.7 mm, vias 2 -> 1
- net GND: track 391.9 -> 390.2 mm
- net Net-(U19-Pad3): track 92.9 -> 91.4 mm, vias 1 -> 0
- net Net-(U17-Pad3): track 22.2 -> 20.8 mm, vias 2 -> 0
- net E0: track 294.5 -> 293.3 mm, vias 8 -> 7
- net NO: track 159.7 -> 158.6 mm
- net X6: track 116.4 -> 115.7 mm, vias 4 -> 3
- net Net-(U19-Pad6): track 75.2 -> 75.7 mm, vias 2 -> 1
- net Net-(U17-Pad6): track 22.5 -> 22.7 mm, vias 2 -> 0
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