File: kicad/memory/memory.kicad_pcb (KiCad board)
At the start: 2 copper layers, 237.5 x 102.9 mm, 55 parts, among them J1 Conn_02x30_Counter_Clockwise, J2 Conn_01x17_Male, J3 Conn_01x17_Male, U1 74LS32, U2 74LS00, U3 74LS32, U4 74LS377, U5 74LS377, U6 28C16, U7 28C16, U8 W24512A, U9 W24512A

Commit message: Fix RAM chip size, add graphics
Parts:
- U8, U9: footprint Package_DIP:DIP-32_W15.24mm_Socket -> Package_DIP:DIP-32_W7.62mm
- moved U9 5.08 mm to (203.2, 121.9)
- moved U8 3.81 mm to (203.2, 78.7)
Routing:
- net A2: track 491.9 -> 555.0 mm, vias 8 -> 12
- net VCC: track 167.8 -> 208.2 mm, vias 7 -> 14
- net A10: track 400.3 -> 388.9 mm, vias 11 -> 8
- net A4: track 475.6 -> 482.5 mm, vias 6 -> 7
- net A6: track 461.5 -> 467.7 mm, vias 6 -> 7
- net D3: track 340.0 -> 334.4 mm
- net D4: track 349.8 -> 344.4 mm
- net D15: track 376.5 -> 371.1 mm
- net D6: track 320.2 -> 325.6 mm
- net D8: track 358.1 -> 363.2 mm, vias 9 -> 10
- net D9: track 357.0 -> 362.0 mm, vias 9 -> 10
- net D10: track 366.5 -> 371.6 mm, vias 8 -> 9
- net A3: track 491.5 -> 496.5 mm, vias 7 -> 8
- net A14: track 390.6 -> 395.7 mm, vias 6 -> 7
- net A1: track 493.3 -> 498.4 mm, vias 8 -> 9
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Other:
- board text added: "Address"
- board text added: "Address register"
- board text added: "Bus"
- board text added: "RAM"
- board text added: "ROM"
- board text added: "ROM/RAM select"
- board text added: "SCAMP Memory Card by jes"

Commit message: Slightly tidy up memory card
Routing:
- net CLK: track 177.7 -> 161.5 mm, vias 2 -> 1
- net GND: track 52.3 -> 63.3 mm, vias 7 -> 8
- net ~AI~: track 204.4 -> 193.9 mm, vias 3 -> 2
- net D9: track 362.0 -> 351.9 mm, vias 10 -> 8
- net A5: track 472.8 -> 463.7 mm, vias 7 -> 5
- net D10: track 371.6 -> 363.6 mm, vias 9 -> 8
- net D8: track 363.2 -> 355.2 mm, vias 10 -> 6
- net Net-(U1-Pad6): track 23.8 -> 30.1 mm, vias 2 -> 1
- net A6: track 467.7 -> 462.3 mm, vias 7 -> 6
- net A14: track 395.7 -> 400.9 mm, vias 7 -> 3
- net A15: track 357.7 -> 352.5 mm, vias 4 -> 1
- net VCC: track 208.2 -> 211.8 mm, vias 14 -> 12
- net D6: track 325.6 -> 322.0 mm, vias 7 -> 6
- net A12: track 396.6 -> 398.7 mm, vias 6 -> 4
- net MI: track 46.3 -> 44.3 mm, vias 1 -> 0
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