File: kicad/instruction/instruction.kicad_pcb (KiCad board)
At the start: 2 copper layers, 237.5 x 102.9 mm, 112 parts, among them J1 Conn_02x30_Counter_Clockwise, J2 Conn_01x17_Male, J3 Conn_01x17_Male, J4 Conn_01x10_Male, J5 Conn_01x15_Male, U1 28C16, U10 74LS161, U11 74LS244, U12 74LS244, U13 74LS161, U14 74LS161, U15 74LS161, U16 74LS161, U17 74LS00, U18 74LS244, U19 74LS244, U2 28C16, U20 74LS244, U21 74LS377, U22 74LS377, U3 74LS04, U4 74LS08, U5 74LS00, U6 74LS08, U7 74LS32, U8 74LS138, U9 74LS138

Commit message: Slightly tidy up instruction card
Routing:
- net CLK: track 274.1 -> 240.2 mm, vias 5 -> 4
- net I1: track 242.4 -> 220.8 mm, vias 7 -> 5
- net GND: track 290.2 -> 277.5 mm
- net GT: track 50.5 -> 44.5 mm, vias 2 -> 0
- net D4: track 118.3 -> 115.0 mm, vias 4 -> 2
- net inv_CLK: track 16.9 -> 14.8 mm, vias 2 -> 0
- net Net-(U5-Pad12): track 15.7 -> 13.8 mm, vias 2 -> 0
- net VCC: track 436.6 -> 438.5 mm, vias 30 -> 31
- net D1: track 136.8 -> 135.2 mm, vias 4 -> 2
- net D6: track 134.4 -> 136.0 mm, vias 6 -> 5
- net I8: track 204.9 -> 203.4 mm
- net D3: track 138.0 -> 139.3 mm, vias 5 -> 4
- net D2: track 127.9 -> 129.0 mm, vias 6 -> 5
- net ~IOH~: track 243.2 -> 242.2 mm, vias 6 -> 5
- net P6: track 29.6 -> 29.1 mm, vias 2 -> 1
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