File: kicad/storage/storage.kicad_pcb (KiCad board)
At the start: 2 copper layers, 12 parts, among them J1 Conn_02x30_Counter_Clockwise, J2 Conn_02x20_Odd_Even, J3 Conn_01x02, J4 Conn_02x20_Odd_Even, J5 Conn_01x02, J6 Conn_01x01, U1 7400, U2 7400, U3 Conn_02x08_Counter_Clockwise

Commit message: Finish storage card
Parts:
- added C4: C, Capacitor_THT:C_Disc_D6.0mm_W2.5mm_P5.00mm, F.Cu at (36.8, 85.2)
- added C5: C, Capacitor_THT:C_Disc_D6.0mm_W2.5mm_P5.00mm, F.Cu at (209.6, 85.2)
- added J7: Conn_01x02, Connector_PinHeader_2.54mm:PinHeader_1x02_P2.54mm_Vertical, F.Cu at (226.0, 106.7)
- added R1: R, Resistor_THT:R_Axial_DIN0207_L6.3mm_D2.5mm_P10.16mm_Horizontal, F.Cu at (240.0, 109.2)
- added R2: R, Resistor_THT:R_Axial_DIN0207_L6.3mm_D2.5mm_P10.16mm_Horizontal, F.Cu at (240.0, 106.7)
- added REF**: MountingHole_3.2mm_M3, MountingHole:MountingHole_3.2mm_M3, F.Cu at (254.0, 33.0)
- added REF**: MountingHole_3.2mm_M3, MountingHole:MountingHole_3.2mm_M3, F.Cu at (254.0, 120.7)
- J2, J4: footprint Connector_PinHeader_2.54mm:PinHeader_2x20_P2.54mm_Vertical -> storage:cfcard
- J6: value Conn_01x01 -> Conn_01x03; footprint Connector_PinHeader_2.54mm:PinHeader_1x01_P2.54mm_Vertical -> Connector_PinHeader_2.54mm:PinHeader_1x03_P2.54mm_Vertical
- moved J3 177.0 mm to (43.2, 87.6)
- moved J2 150.7 mm to (55.0, 44.5)
- moved J6 132.5 mm to (243.8, 111.8), turned to 180 degrees
- moved U3 116.7 mm to (174.0, 97.8)
- moved U2 83.7 mm to (152.4, 100.3)
- moved C3 78.4 mm to (180.3, 92.7), turned to 180 degrees
- moved U1 77.7 mm to (130.8, 100.3)
- moved C2 71.8 mm to (158.8, 95.2), turned to 180 degrees
- moved C1 65.0 mm to (137.2, 95.2), turned to 180 degrees
- moved J4 57.9 mm to (228.0, 44.5)
- moved J1 43.7 mm to (26.7, 40.0)
- moved J5 10.7 mm to (215.9, 87.6)
Connections:
- J1 pad 38: (no net) -> WR
- J6 pad 1: WR -> GND
Routing:
- net ~RESET~: track 0.00 -> 237.4 mm, vias 0 -> 1
- net A2: track 0.00 -> 235.3 mm, vias 0 -> 1
- net A1: track 0.00 -> 234.3 mm, vias 0 -> 1
- net A0: track 0.00 -> 231.8 mm, vias 0 -> 1
- net D1: track 0.00 -> 227.9 mm, vias 0 -> 2
- net D0: track 0.00 -> 227.9 mm, vias 0 -> 2
- net D3: track 0.00 -> 221.4 mm, vias 0 -> 2
- net D2: track 0.00 -> 221.0 mm, vias 0 -> 2
- net D4: track 0.00 -> 213.1 mm, vias 0 -> 2
- net D5: track 0.00 -> 212.3 mm, vias 0 -> 2
- net ~IOWR~: track 0.00 -> 211.9 mm, vias 0 -> 1
- net D7: track 0.00 -> 209.8 mm, vias 0 -> 1
- net D15: track 0.00 -> 207.8 mm
- net D9: track 0.00 -> 206.9 mm
- net D13: track 0.00 -> 206.7 mm
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- added copper zone on F.Cu, net GND
- added copper zone on B.Cu, net VCC
Other:
- board outline added: 237.5 x 102.9 mm
- board text added: "GND"
- board text added: "SCAMP Storage Card by jes"
- board text added: "VCC"
