File: kicad/storage/storage.kicad_pcb (KiCad board)
At the start: 2 copper layers, 237.5 x 102.9 mm, 19 parts, among them J1 Conn_02x30_Counter_Clockwise, J2 Conn_02x20_Odd_Even, J3 Conn_01x02, J4 Conn_02x20_Odd_Even, J5 Conn_01x02, J6 Conn_01x03, J7 Conn_01x02, U1 7400, U2 7400, U3 Conn_02x08_Counter_Clockwise

Commit message: Add 74HCT245 bus transceivers to storage card
Parts:
- added C6: C, Capacitor_THT:C_Disc_D6.0mm_W2.5mm_P5.00mm, F.Cu at (69.8, 75.0)
- added C7: C, Capacitor_THT:C_Disc_D6.0mm_W2.5mm_P5.00mm, F.Cu at (96.5, 86.4)
- added C8: C, Capacitor_THT:C_Disc_D6.0mm_W2.5mm_P5.00mm, F.Cu at (210.8, 91.5)
- added U4: 74HC245, Package_DIP:DIP-20_W7.62mm_Socket, F.Cu at (47.0, 39.4)
- added U5: 74HC245, Package_DIP:DIP-20_W7.62mm_Socket, F.Cu at (47.0, 54.6)
- added U6: 74LS08, Package_DIP:DIP-14_W7.62mm_Socket, F.Cu at (74.9, 81.3)
- moved C5 171.6 mm to (41.9, 48.3)
- moved C3 142.1 mm to (39.4, 74.9), turned to 270 degrees
- moved U3 130.6 mm to (44.5, 81.3), turned to 90 degrees
- moved C1 97.9 mm to (39.4, 100.3), turned to 270 degrees
- moved C2 89.0 mm to (69.8, 100.3), turned to 270 degrees
- moved U1 86.6 mm to (44.5, 106.7), turned to 90 degrees
- moved U2 77.7 mm to (74.9, 106.7), turned to 90 degrees
- moved J2 58.7 mm to (113.7, 44.5)
- moved J3 58.4 mm to (101.6, 87.6)
- moved C4 52.4 mm to (41.9, 33.0)
- moved J5 5.08 mm to (215.9, 92.7)
- moved J7 0.54 mm to (225.4, 106.7)
Connections:
- J1 pad 17: (no net) -> /Z
- J1 pad 18: (no net) -> /LT
- J1 pad 19: (no net) -> /~EO~
- J1 pad 20: (no net) -> /~XI~
- J1 pad 21: (no net) -> /~YI~
- J1 pad 22: (no net) -> /~AI~
- J1 pad 23: (no net) -> /MO
- J1 pad 24: (no net) -> /MI
- J1 pad 26: (no net) -> /DI
- J1 pad 27: (no net) -> Net-(J1-Pad27)
- J1 pad 29: (no net) -> /CLK
- J1 pad 32: (no net) -> Net-(J1-Pad32)
- J1 pad 33: (no net) -> Net-(J1-Pad33)
- J1 pad 34: (no net) -> Net-(J1-Pad34)
- J1 pad 35: (no net) -> Net-(J1-Pad35)
- J1 pad 36: (no net) -> Net-(J1-Pad36)
- J1 pad 37: (no net) -> Net-(J1-Pad37)
- J1 pad 39: (no net) -> /NO
- J1 pad 40: (no net) -> /F
- J1 pad 41: (no net) -> /NY
- J1 pad 42: (no net) -> /EY
- J1 pad 43: (no net) -> /NX
- J1 pad 44: (no net) -> /EX
- J1 pad 45: (no net) -> /A15
- J1 pad 46: (no net) -> /A14
- J1 pad 47: (no net) -> /A13
- J1 pad 48: (no net) -> /A12
- J1 pad 49: (no net) -> /A11
- J1 pad 50: (no net) -> /A10
- J1 pad 51: (no net) -> /A9
- J1 pad 53: (no net) -> /A7
- J2 pad 10: D11 -> 245D11
- J2 pad 11: D3 -> 245D3
- J2 pad 12: D12 -> 245D12
- J2 pad 13: D2 -> 245D2
- J2 pad 14: D13 -> 245D13
- J2 pad 15: D1 -> 245D1
- J2 pad 16: D14 -> 245D14
- J2 pad 17: D0 -> 245D0
- J2 pad 18: D15 -> 245D15
- J2 pad 20: (no net) -> Net-(J2-Pad20)
- J2 pad 21: (no net) -> Net-(J2-Pad21)
- J2 pad 27: (no net) -> Net-(J2-Pad27)
- J2 pad 28: (no net) -> Net-(J2-Pad28)
- J2 pad 29: (no net) -> Net-(J2-Pad29)
- J2 pad 3: D7 -> 245D7
- J2 pad 31: (no net) -> Net-(J2-Pad31)
- J2 pad 32: (no net) -> Net-(J2-Pad32)
- J2 pad 34: (no net) -> Net-(J2-Pad34)
- J2 pad 39: (no net) -> Net-(J2-Pad39)
- J2 pad 4: D8 -> 245D8
- J2 pad 5: D6 -> 245D6
- J2 pad 6: D9 -> 245D9
- J2 pad 7: D5 -> 245D5
- J2 pad 8: D10 -> 245D10
- J2 pad 9: D4 -> 245D4
- J4 pad 10: D11 -> 245D11
- J4 pad 11: D3 -> 245D3
- J4 pad 12: D12 -> 245D12
- J4 pad 13: D2 -> 245D2
- J4 pad 14: D13 -> 245D13
- J4 pad 15: D1 -> 245D1
- J4 pad 16: D14 -> 245D14
- J4 pad 17: D0 -> 245D0
- J4 pad 18: D15 -> 245D15
- J4 pad 20: (no net) -> Net-(J4-Pad20)
- J4 pad 21: (no net) -> Net-(J4-Pad21)
- J4 pad 27: (no net) -> Net-(J4-Pad27)
- J4 pad 28: (no net) -> Net-(J4-Pad28)
- J4 pad 29: (no net) -> Net-(J4-Pad29)
- J4 pad 3: D7 -> 245D7
- J4 pad 31: (no net) -> Net-(J4-Pad31)
- J4 pad 32: (no net) -> Net-(J4-Pad32)
- J4 pad 34: (no net) -> Net-(J4-Pad34)
- J4 pad 39: (no net) -> Net-(J4-Pad39)
- J4 pad 4: D8 -> 245D8
- J4 pad 5: D6 -> 245D6
- J4 pad 6: D9 -> 245D9
- J4 pad 7: D5 -> 245D5
- J4 pad 8: D10 -> 245D10
- J4 pad 9: D4 -> 245D4
- J6 pad 1: GND -> VCC
- U2 pad 10: (no net) -> Net-(U2-Pad10)
- U2 pad 11: (no net) -> Net-(U2-Pad11)
- U2 pad 12: (no net) -> Net-(U2-Pad12)
- U2 pad 13: (no net) -> Net-(U2-Pad13)
- U2 pad 8: (no net) -> Net-(U2-Pad8)
- U2 pad 9: (no net) -> Net-(U2-Pad9)
Routing:
- net 245D8: track 0.00 -> 313.1 mm
- net 245D0: track 0.00 -> 207.5 mm, vias 0 -> 2
- net D0: track 227.9 -> 23.6 mm, vias 2 -> 0
- net 245D1: track 0.00 -> 203.8 mm, vias 0 -> 2
- net 245D2: track 0.00 -> 198.9 mm, vias 0 -> 2
- net D1: track 227.9 -> 29.8 mm, vias 2 -> 0
- net 245D3: track 0.00 -> 194.3 mm, vias 0 -> 2
- net D2: track 221.0 -> 29.3 mm, vias 2 -> 0
- net 245D4: track 0.00 -> 189.8 mm, vias 0 -> 2
- net D3: track 221.4 -> 36.0 mm, vias 2 -> 0
- net 245D5: track 0.00 -> 185.1 mm, vias 0 -> 2
- net 245D6: track 0.00 -> 180.4 mm, vias 0 -> 2
- net 245D9: track 0.00 -> 178.2 mm
- net D4: track 213.1 -> 36.0 mm, vias 2 -> 0
- net D8: track 203.6 -> 26.9 mm
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Other:
- board text added: "Rev B"
